Commit message: can resize

File: urdf/conveyor_belt.urdf.xacro (robot description, xacro)
@@ -6,4 +6,6 @@
   <xacro:arg name="namespace" default="belt1"/>
   <xacro:arg name="max_velocity" default="0.3"/>
+  <xacro:arg name="scale" default="0.25"/>
+  <xacro:property name="sc" value="$(arg scale)"/>
   <xacro:macro name="body_color">
     <visual>
@@ -48,5 +50,6 @@
       <geometry>
         <mesh
-          filename="package://conveyor_belt/meshes/base_link.STL" />
+          filename="package://conveyor_belt/meshes/base_link.STL"
+          scale="${sc} ${sc} ${sc}" />
       </geometry>
       <material
@@ -62,5 +65,6 @@
       <geometry>
         <mesh
-          filename="package://conveyor_belt/meshes/base_link.STL" />
+          filename="package://conveyor_belt/meshes/base_link.STL"
+          scale="${sc} ${sc} ${sc}" />
       </geometry>
     </collision>
@@ -70,5 +74,5 @@
     <inertial>
       <origin
-        xyz="2.84 0.00499999999999995 2.76334119905601E-17"
+        xyz="${2.84 * sc} ${0.005 * sc} 0"
         rpy="0 0 0" />
       <mass
@@ -88,5 +92,6 @@
       <geometry>
         <mesh
-          filename="package://conveyor_belt/meshes/belt_link.STL" />
+          filename="package://conveyor_belt/meshes/belt_link.STL"
+          scale="${sc} ${sc} ${sc}" />
       </geometry>
       <material
@@ -102,5 +107,6 @@
       <geometry>
         <mesh
-          filename="package://conveyor_belt/meshes/belt_link.STL" />
+          filename="package://conveyor_belt/meshes/belt_link.STL"
+          scale="${sc} ${sc} ${sc}" />
       </geometry>
     </collision>
@@ -110,5 +116,5 @@
     type="prismatic">
     <origin
-      xyz="-2.83 0 0.3"
+      xyz="${-2.83 * sc} 0 ${0.3 * sc}"
       rpy="1.5708 0 0" />
     <parent
