Commit message: resize box

File: urdf/box.urdf.xacro (robot description, xacro)
@@ -4,4 +4,6 @@
      For more information, please see http://wiki.ros.org/sw_urdf_exporter -->
 <robot  name="box" xmlns:xacro="http://ros.org/wiki/xacro">
+  <xacro:arg name="scale" default="1.0"/>
+  <xacro:property name="sc" value="$(arg scale)"/>
   <xacro:macro name="body_color">
     <visual>
@@ -46,5 +48,6 @@
       <geometry>
         <mesh
-          filename="package://conveyor_belt/meshes/box/base_link.STL" />
+          filename="package://conveyor_belt/meshes/box/base_link.STL"
+          scale="${sc} ${sc} ${sc}" />
       </geometry>
       <material
@@ -60,5 +63,6 @@
       <geometry>
         <mesh
-          filename="package://conveyor_belt/meshes/box/base_link.STL" />
+          filename="package://conveyor_belt/meshes/box/base_link.STL"
+          scale="${sc} ${sc} ${sc}" />
       </geometry>
     </collision>
@@ -86,5 +90,6 @@
       <geometry>
         <mesh
-          filename="package://conveyor_belt/meshes/box/lid_link.STL" />
+          filename="package://conveyor_belt/meshes/box/lid_link.STL"
+          scale="${sc} ${sc} ${sc}" />
       </geometry>
       <material
@@ -100,5 +105,6 @@
       <geometry>
         <mesh
-          filename="package://conveyor_belt/meshes/box/lid_link.STL" />
+          filename="package://conveyor_belt/meshes/box/lid_link.STL"
+          scale="${sc} ${sc} ${sc}" />
       </geometry>
     </collision>
@@ -108,5 +114,5 @@
     type="fixed">
     <origin
-      xyz="0.018291 0.015197 0.16816"
+      xyz="${0.018291 * sc} ${0.015197 * sc} ${0.16816 * sc}"
       rpy="-1.5708 0 3.1416" />
     <parent
